File: hardware/Nixie_clock/Nixie_clock.kicad_sch (KiCad schematic)
At the start: 76 parts, among them J1 90814-0912, J10 Conn_01x02_Pin, J11 12V_IN, J12 UART, J13 Conn_01x02_Pin, J14 Debug1, J16 Debug, J2 90814-0912, J3 90814-0912, J4 90814-0912, J5 90814-0912, J6 90814-0912, J7 90814-0912, J8 90814-0912, J9 Conn_01x02_Pin, Q1 PMV37ENEAR, Q2 PMV37ENEAR, Q3 PMV37ENEAR, Q4 PMV37ENEAR, Q5 PMV37ENEAR, SW1 Tog_ON_ON_(ON), U1 MAX1771xSA, U2 ESP32-C3-MINI-1, U3 TLV76133DCY, Y1 AIUR-08 coil

Commit message: Hardware revision 1.1
Fix: HV5622 pad spacing, use bigger DCDC FET, add LS NFETs PD resistors, Minor layout fixes.
Parts:
- removed C2: 10u, Capacitor_SMD:C_1206_3216Metric_Pad1.33x1.80mm_HandSolder, symbol Device:C
- removed Q1: PMV37ENEAR, PMV37ENEAR:SOT95P230X110-3N, symbol PMV37ENEAR:PMV37ENEAR
- added J16: Conn_01x02_Pin, Connector_PinHeader_2.54mm:PinHeader_1x02_P2.54mm_Vertical, symbol Connector:Conn_01x02_Pin
- added Q1: IPD60R280P7, Package_TO_SOT_SMD:TO-252-2, symbol Transistor_FET:IPD50R380CE
- added R24, R25, R26: 10k, Resistor_SMD:R_1206_3216Metric_Pad1.30x1.75mm_HandSolder, symbol Device:R
- added R27: 3.6k, Resistor_SMD:R_1206_3216Metric_Pad1.30x1.75mm_HandSolder, symbol Device:R
- C16: renamed from C13; value 0.1u -> 10nF
- J10: renamed from J9; value Conn_01x02_Pin -> HV_EN
- J13: value Conn_01x02_Pin -> 3.3V_EN
- R17, R18, R19, R20: value 10k -> 4.7k
- Y1: value AIUR-08 coil -> 100uH
- renumbered C10 to C1, C7 to C10, C8 to C11, C9 to C12, C16 to C13, C12 to C14, C11 to C15, C14 to C2, C15 to C3, C1 to C4, C3 to C6, C4 to C7, C5 to C8, C6 to C9, J10 to J11, J14 to J12, J11 to J14, J12 to J15, J16 to J9, R24 to R28, R25 to R29, R26 to R30, R27 to R31, R28 to R32, U3 to U2, U2 to U3
Connections:
- net +12V: now also J16.2 (Pin_2)
- net GND: now also J16.1 (Pin_1), R24.2, R25.2, R26.2, R27.2
- net at D1.2 (A), Y1.4: now also Q1.2 (D)
- net at U1.1 (EXT): now also Q1.1 (G)
- net at R23.1, U1.8 (CS): now also Q1.3 (S)
- net LS1_in renamed LS_data_in
- net LS_data_in: now also R25.1
- net LS1_out renamed LS_data_out
- net LS2_in renamed LS_clk_in
- net LS_clk_in: now also R24.1
- net LS2_out renamed LS_clk_out
- net LS3_in renamed LS_LE_in
- net LS_LE_in: now also R26.1
- net LS3_out renamed LS_LE_out
- net LS4_in renamed LS_BL_in
- net LS_BL_in: now also R27.1
- net LS4_out renamed LS_BL_out
- no-connect marks 22 -> 20
Other:
- moved on the sheet: C4, C6, J10, J12, Q2, Q3, Q4, R17
